File: amp.sch (KiCad schematic (older format))
At the start: 25 parts, among them Q2 MMBF170, Q3 IRF510, Q4 IRF510, T1 8:8, T2 8:8, T3 2:3

Commit message: Finished band filters schematic
- Associated last of the capacitors with footprints
- Associated inductors
Parts:
- C15, C16, C17: footprint (none) -> Capacitors_SMD:C_0805_HandSoldering
- JP1: footprint (none) -> Pin_Headers:Pin_Header_Straight_1x02
- Q2: footprint (none) -> Transistors_SMD:sot23
- Q3, Q4: footprint (none) -> Transistors_TO-220:TO-220_FET-GDS_Vertical_LargePads
- R11, R12, R14, R15, R5, R6, R8: footprint (none) -> Discret:R1
- RV1, RV2: footprint (none) -> nu9j-footprints:Potentiometer_Trimmer_Piher_PT10_H01
- T1, T2: footprint (none) -> nu9j-footprints:BN2-202
- T3: footprint (none) -> nu9j-footprints:BN2-3312
Changed lines of the file:
@@
 F 0 "T2" H 7750 4950 70  0000 C CNN
 F 1 "8:8" H 7750 4400 70  0000 C CNN
-F 2 "" H 7750 4700 60  0001 C CNN
+F 2 "nu9j-footprints:BN2-202" H 7750 4700 60  0001 C CNN
 F 3 "" H 7750 4700 60  0000 C CNN
 	1    7750 4700
@@
 F 0 "T3" H 8900 4950 70  0000 C CNN
 F 1 "2:3" H 8900 4400 70  0000 C CNN
-F 2 "" H 8900 4700 60  0001 C CNN
+F 2 "nu9j-footprints:BN2-3312" H 8900 4700 60  0001 C CNN
 F 3 "" H 8900 4700 60  0000 C CNN
 	1    8900 4700
@@
 F 0 "T1" H 5000 5100 70  0000 C CNN
 F 1 "8:8" H 5000 4550 70  0000 C CNN
-F 2 "" H 5000 4850 60  0001 C CNN
+F 2 "nu9j-footprints:BN2-202" H 5000 4850 60  0001 C CNN
 F 3 "" H 5000 4850 60  0000 C CNN
 	1    5000 4850
@@
 F 0 "Q3" H 7010 4470 60  0000 R CNN
 F 1 "IRF510" H 7010 4150 60  0000 R CNN
-F 2 "" H 7000 4300 60  0001 C CNN
+F 2 "Transistors_TO-220:TO-220_FET-GDS_Vertical_LargePads" H 7000 4300 60  0001 C CNN
 F 3 "" H 7000 4300 60  0000 C CNN
 	1    7000 4300
@@
 F 0 "Q4" H 7010 5570 60  0000 R CNN
 F 1 "IRF510" H 7010 5250 60  0000 R CNN
-F 2 "" H 7000 5400 60  0001 C CNN
+F 2 "Transistors_TO-220:TO-220_FET-GDS_Vertical_LargePads" H 7000 5400 60  0001 C CNN
 F 3 "" H 7000 5400 60  0000 C CNN
 	1    7000 5400
@@
 F 0 "R5" V 3580 4700 40  0000 C CNN
 F 1 "300" V 3507 4701 40  0000 C CNN
-F 2 "" V 3430 4700 30  0001 C CNN
+F 2 "Discret:R1" V 3430 4700 30  0001 C CNN
 F 3 "" H 3500 4700 30  0000 C CNN
 	1    3500 4700
@@
 F 0 "R6" V 3980 4450 40  0000 C CNN
 F 1 "18" V 3907 4451 40  0000 C CNN
-F 2 "" V 3830 4450 30  0001 C CNN
+F 2 "Discret:R1" V 3830 4450 30  0001 C CNN
 F 3 "" H 3900 4450 30  0000 C CNN
 	1    3900 4450
@@
 F 0 "R8" V 4330 4700 40  0000 C CNN
 F 1 "300" V 4257 4701 40  0000 C CNN
-F 2 "" V 4180 4700 30  0001 C CNN
+F 2 "Discret:R1" V 4180 4700 30  0001 C CNN
 F 3 "" H 4250 4700 30  0000 C CNN
 	1    4250 4700
@@
 F 0 "R11" V 5680 4550 40  0000 C CNN
 F 1 "51" V 5607 4551 40  0000 C CNN
-F 2 "" V 5530 4550 30  0001 C CNN
+F 2 "Discret:R1" V 5530 4550 30  0001 C CNN
 F 3 "" H 5600 4550 30  0000 C CNN
 	1    5600 4550
@@
 F 0 "R14" V 5880 4550 40  0000 C CNN
 F 1 "51" V 5807 4551 40  0000 C CNN
-F 2 "" V 5730 4550 30  0001 C CNN
+F 2 "Discret:R1" V 5730 4550 30  0001 C CNN
 F 3 "" H 5800 4550 30  0000 C CNN
 	1    5800 4550
@@
 F 0 "R12" V 5680 5150 40  0000 C CNN
 F 1 "51" V 5607 5151 40  0000 C CNN
-F 2 "" V 5530 5150 30  0001 C CNN
+F 2 "Discret:R1" V 5530 5150 30  0001 C CNN
 F 3 "" H 5600 5150 30  0000 C CNN
 	1    5600 5150
@@
 F 0 "R15" V 5880 5150 40  0000 C CNN
 F 1 "51" V 5807 5151 40  0000 C CNN
-F 2 "" V 5730 5150 30  0001 C CNN
+F 2 "Discret:R1" V 5730 5150 30  0001 C CNN
 F 3 "" H 5800 5150 30  0000 C CNN
 	1    5800 5150
@@
 F 0 "C15" H 6000 4400 40  0000 L CNN
 F 1 "0.1u" H 6006 4215 40  0000 L CNN
-F 2 "" H 6038 4150 30  0001 C CNN
+F 2 "Capacitors_SMD:C_0805_HandSoldering" H 6038 4150 30  0001 C CNN
 F 3 "" H 6000 4300 60  0000 C CNN
 	1    6000 4300
@@
 F 0 "C16" H 6000 5500 40  0000 L CNN
 F 1 "0.1u" H 6006 5315 40  0000 L CNN
-F 2 "" H 6038 5250 30  0001 C CNN
+F 2 "Capacitors_SMD:C_0805_HandSoldering" H 6038 5250 30  0001 C CNN
 F 3 "" H 6000 5400 60  0000 C CNN
 	1    6000 5400
@@
 	2950 4450 3650 4450
 $Comp
-L GND #PWR44
+L GND #PWR040
 U 1 1 5470F4C6
 P 4800 5250
-F 0 "#PWR44" H 4800 5250 30  0001 C CNN
+F 0 "#PWR040" H 4800 5250 30  0001 C CNN
 F 1 "GND" H 4800 5180 30  0001 C CNN
 F 2 "" H 4800 5250 60  0000 C CNN
@@
 $EndComp
 $Comp
-L GND #PWR42
+L GND #PWR041
 U 1 1 5470F4DA
 P 4250 5250
-F 0 "#PWR42" H 4250 5250 30  0001 C CNN
+F 0 "#PWR041" H 4250 5250 30  0001 C CNN
 F 1 "GND" H 4250 5180 30  0001 C CNN
 F 2 "" H 4250 5250 60  0000 C CNN
@@
 $EndComp
 $Comp
-L GND #PWR40
+L GND #PWR042
 U 1 1 5470F4EE
 P 3500 5250
-F 0 "#PWR40" H 3500 5250 30  0001 C CNN
+F 0 "#PWR042" H 3500 5250 30  0001 C CNN
 F 1 "GND" H 3500 5180 30  0001 C CNN
 F 2 "" H 3500 5250 60  0000 C CNN
@@
 Connection ~ 7350 3950
 $Comp
-L GND #PWR47
+L GND #PWR043
 U 1 1 5470F5FC
 P 7100 4500
-F 0 "#PWR47" H 7100 4500 30  0001 C CNN
+F 0 "#PWR043" H 7100 4500 30  0001 C CNN
 F 1 "GND" H 7100 4430 30  0001 C CNN
 F 2 "" H 7100 4500 60  0000 C CNN
@@
 $EndComp
 $Comp
-L GND #PWR48
+L GND #PWR044
 U 1 1 5470F610
 P 7150 5600
-F 0 "#PWR48" H 7150 5600 30  0001 C CNN
+F 0 "#PWR044" H 7150 5600 30  0001 C CNN
 F 1 "GND" H 7150 5530 30  0001 C CNN
 F 2 "" H 7150 5600 60  0000 C CNN
@@
 amp_in
 $Comp
-L GND #PWR51
+L GND #PWR045
 U 1 1 5470F625
 P 9300 5200
-F 0 "#PWR51" H 9300 5200 30  0001 C CNN
+F 0 "#PWR045" H 9300 5200 30  0001 C CNN
 F 1 "GND" H 9300 5130 30  0001 C CNN
 F 2 "" H 9300 5200 60  0000 C CNN
@@
 F 0 "RV1" H 4150 2350 50  0000 C CNN
 F 1 "5k" H 4150 2450 50  0000 C CNN
-F 2 "" H 4150 2450 60  0001 C CNN
+F 2 "nu9j-footprints:Potentiometer_Trimmer_Piher_PT10_H01" H 4150 2450 60  0001 C CNN
 F 3 "" H 4150 2450 60  0000 C CNN
 	1    4150 2450
@@
 F 0 "RV2" H 5350 2350 50  0000 C CNN
 F 1 "5k" H 5350 2450 50  0000 C CNN
-F 2 "" H 5350 2450 60  0001 C CNN
+F 2 "nu9j-footprints:Potentiometer_Trimmer_Piher_PT10_H01" H 5350 2450 60  0001 C CNN
 F 3 "" H 5350 2450 60  0000 C CNN
 	1    5350 2450
@@
 $EndComp
 $Comp
-L +5V #PWR41
+L +5V #PWR046
 U 1 1 5470F81B
 P 4150 2200
-F 0 "#PWR41" H 4150 2290 20  0001 C CNN
+F 0 "#PWR046" H 4150 2290 20  0001 C CNN
 F 1 "+5V" H 4150 2290 30  0000 C CNN
 F 2 "" H 4150 2200 60  0000 C CNN
@@
 $EndComp
 $Comp
-L GND #PWR43
+L GND #PWR047
 U 1 1 5470F84C
 P 4750 3700
-F 0 "#PWR43" H 4750 3700 30  0001 C CNN
+F 0 "#PWR047" H 4750 3700 30  0001 C CNN
 F 1 "GND" H 4750 3630 30  0001 C CNN
 F 2 "" H 4750 3700 60  0000 C CNN
@@
 vb2
 $Comp
-L +12V #PWR49
+L +12V #PWR048
 U 1 1 5470F9E0
 P 7350 3750
-F 0 "#PWR49" H 7350 3700 20  0001 C CNN
+F 0 "#PWR048" H 7350 3700 20  0001 C CNN
 F 1 "+12V" H 7350 3850 30  0000 C CNN
 F 2 "" H 7350 3750 60  0000 C CNN
@@
 F 0 "C17" H 7550 3850 40  0000 L CNN
 F 1 "0.1u" H 7556 3665 40  0000 L CNN
-F 2 "" H 7588 3600 30  0001 C CNN
+F 2 "Capacitors_SMD:C_0805_HandSoldering" H 7588 3600 30  0001 C CNN
 F 3 "" H 7550 3750 60  0000 C CNN
 	1    7550 3750
@@
 $EndComp
 $Comp
-L GND #PWR50
+L GND #PWR049
 U 1 1 5470FA0D
 P 7750 3750
-F 0 "#PWR50" H 7750 3750 30  0001 C CNN
+F 0 "#PWR049" H 7750 3750 30  0001 C CNN
 F 1 "GND" H 7750 3680 30  0001 C CNN
 F 2 "" H 7750 3750 60  0000 C CNN
@@
 $EndComp
 $Comp
-L GND #PWR46
+L GND #PWR050
 U 1 1 5470FB98
 P 6400 4850
-F 0 "#PWR46" H 6400 4850 30  0001 C CNN
+F 0 "#PWR050" H 6400 4850 30  0001 C CNN
 F 1 "GND" H 6400 4780 30  0001 C CNN
 F 2 "" H 6400 4850 60  0000 C CNN
@@
 F 0 "JP1" H 6100 5000 60  0000 C CNN
 F 1 "AMP_BAL" H 6100 4770 40  0000 C CNN
-F 2 "" H 6100 4850 60  0001 C CNN
+F 2 "Pin_Headers:Pin_Header_Straight_1x02" H 6100 4850 60  0001 C CNN
 F 3 "" H 6100 4850 60  0000 C CNN
 	1    6100 4850
@@
 F 0 "Q2" H 4660 3670 60  0000 R CNN
 F 1 "MMBF170" H 4660 3350 60  0000 R CNN
-F 2 "" H 4650 3500 60  0001 C CNN
+F 2 "Transistors_SMD:sot23" H 4650 3500 60  0001 C CNN
 F 3 "" H 4650 3500 60  0000 C CNN
 	1    4650 3500
@@
 Connection ~ 4750 3200
 $Comp
-L +5V #PWR45
+L +5V #PWR051
 U 1 1 5470FCA2
 P 5350 2200
-F 0 "#PWR45" H 5350 2290 20  0001 C CNN
+F 0 "#PWR051" H 5350 2290 20  0001 C CNN
 F 1 "+5V" H 5350 2290 30  0000 C CNN
 F 2 "" H 5350 2200 60  0000 C CNN

Commit message: Fixed pin assignment issues in pcb layout
Parts:
- Q2: footprint Transistors_SMD:sot23 -> nu9j-footprints:sot23-DGS
Changed lines of the file:
@@
 F 0 "Q2" H 4660 3670 60  0000 R CNN
 F 1 "MMBF170" H 4660 3350 60  0000 R CNN
-F 2 "Transistors_SMD:sot23" H 4650 3500 60  0001 C CNN
+F 2 "nu9j-footprints:sot23-DGS" H 4650 3500 60  0001 C CNN
 F 3 "" H 4650 3500 60  0000 C CNN
 	1    4650 3500
