File: amp.sch (KiCad schematic (older format))
At the start: 25 parts, among them Q3 IRF510, Q4 IRF510, T1 8:8, T2 8:8, T3 2:3, U5 LTV-356T

Commit message: Update project to kicad bzr 6336
I guess some parts are now outdated
Parts:
- C15, C16, C17: symbol C -> C-RESCUE-qrpamp
- R10, R11, R12, R13, R14, R15, R16, R17, R18, R5, R6, R7, R8, R9: symbol R -> R-RESCUE-qrpamp
Changed lines of the file:
@@
 EESchema Schematic File Version 2
+LIBS:qrpamp-rescue
 LIBS:power
 LIBS:device
@@
 $EndComp
 $Comp
-L R R5
+L R-RESCUE-qrpamp R5
 U 1 1 5470F3E3
 P 3500 4700
+AR Path="/5470F3E3" Ref="R5"  Part="1"
+AR Path="/5470C606/5470F3E3" Ref="R5"  Part="1"
 F 0 "R5" V 3580 4700 40  0000 C CNN
 F 1 "300" V 3507 4701 40  0000 C CNN
@@
 $EndComp
 $Comp
-L R R6
+L R-RESCUE-qrpamp R6
 U 1 1 5470F3F5
 P 3900 4450
+AR Path="/5470F3F5" Ref="R6"  Part="1"
+AR Path="/5470C606/5470F3F5" Ref="R6"  Part="1"
 F 0 "R6" V 3980 4450 40  0000 C CNN
 F 1 "18" V 3907 4451 40  0000 C CNN
@@
 $EndComp
 $Comp
-L R R8
+L R-RESCUE-qrpamp R8
 U 1 1 5470F400
 P 4250 4700
+AR Path="/5470F400" Ref="R8"  Part="1"
+AR Path="/5470C606/5470F400" Ref="R8"  Part="1"
 F 0 "R8" V 4330 4700 40  0000 C CNN
 F 1 "300" V 4257 4701 40  0000 C CNN
@@
 $EndComp
 $Comp
-L R R11
+L R-RESCUE-qrpamp R11
 U 1 1 5470F415
 P 5600 4550
+AR Path="/5470F415" Ref="R11"  Part="1"
+AR Path="/5470C606/5470F415" Ref="R11"  Part="1"
 F 0 "R11" V 5680 4550 40  0000 C CNN
 F 1 "51" V 5607 4551 40  0000 C CNN
@@
 $EndComp
 $Comp
-L R R14
+L R-RESCUE-qrpamp R14
 U 1 1 5470F420
 P 5800 4550
+AR Path="/5470F420" Ref="R14"  Part="1"
+AR Path="/5470C606/5470F420" Ref="R14"  Part="1"
 F 0 "R14" V 5880 4550 40  0000 C CNN
 F 1 "51" V 5807 4551 40  0000 C CNN
@@
 $EndComp
 $Comp
-L R R12
+L R-RESCUE-qrpamp R12
 U 1 1 5470F42B
 P 5600 5150
+AR Path="/5470F42B" Ref="R12"  Part="1"
+AR Path="/5470C606/5470F42B" Ref="R12"  Part="1"
 F 0 "R12" V 5680 5150 40  0000 C CNN
 F 1 "51" V 5607 5151 40  0000 C CNN
@@
 $EndComp
 $Comp
-L R R15
+L R-RESCUE-qrpamp R15
 U 1 1 5470F436
 P 5800 5150
+AR Path="/5470F436" Ref="R15"  Part="1"
+AR Path="/5470C606/5470F436" Ref="R15"  Part="1"
 F 0 "R15" V 5880 5150 40  0000 C CNN
 F 1 "51" V 5807 5151 40  0000 C CNN
@@
 $EndComp
 $Comp
-L C C15
+L C-RESCUE-qrpamp C15
 U 1 1 5470F443
 P 6000 4300
+AR Path="/5470F443" Ref="C15"  Part="1"
+AR Path="/5470C606/5470F443" Ref="C15"  Part="1"
 F 0 "C15" H 6000 4400 40  0000 L CNN
 F 1 "0.1u" H 6006 4215 40  0000 L CNN
@@
 $EndComp
 $Comp
-L C C16
+L C-RESCUE-qrpamp C16
 U 1 1 5470F455
 P 6000 5400
+AR Path="/5470F455" Ref="C16"  Part="1"
+AR Path="/5470C606/5470F455" Ref="C16"  Part="1"
 F 0 "C16" H 6000 5500 40  0000 L CNN
 F 1 "0.1u" H 6006 5315 40  0000 L CNN
@@
 $EndComp
 $Comp
-L R R16
+L R-RESCUE-qrpamp R16
 U 1 1 5470F460
 P 6550 4300
+AR Path="/5470F460" Ref="R16"  Part="1"
+AR Path="/5470C606/5470F460" Ref="R16"  Part="1"
 F 0 "R16" V 6630 4300 40  0000 C CNN
 F 1 "10" V 6557 4301 40  0000 C CNN
@@
 $EndComp
 $Comp
-L R R17
+L R-RESCUE-qrpamp R17
 U 1 1 5470F475
 P 6550 5400
+AR Path="/5470F475" Ref="R17"  Part="1"
+AR Path="/5470C606/5470F475" Ref="R17"  Part="1"
 F 0 "R17" V 6630 5400 40  0000 C CNN
 F 1 "10" V 6557 5401 40  0000 C CNN
@@
 	2950 4450 3650 4450
 $Comp
-L GND #PWR048
+L GND-RESCUE-qrpamp #PWR048
 U 1 1 5470F4C6
 P 4800 5250
+AR Path="/5470F4C6" Ref="#PWR048"  Part="1"
+AR Path="/5470C606/5470F4C6" Ref="#PWR048"  Part="1"
 F 0 "#PWR048" H 4800 5250 30  0001 C CNN
 F 1 "GND" H 4800 5180 30  0001 C CNN
@@
 $EndComp
 $Comp
-L GND #PWR049
+L GND-RESCUE-qrpamp #PWR049
 U 1 1 5470F4DA
 P 4250 5250
+AR Path="/5470F4DA" Ref="#PWR049"  Part="1"
+AR Path="/5470C606/5470F4DA" Ref="#PWR049"  Part="1"
 F 0 "#PWR049" H 4250 5250 30  0001 C CNN
 F 1 "GND" H 4250 5180 30  0001 C CNN
@@
 $EndComp
 $Comp
-L GND #PWR050
+L GND-RESCUE-qrpamp #PWR050
 U 1 1 5470F4EE
 P 3500 5250
+AR Path="/5470F4EE" Ref="#PWR050"  Part="1"
+AR Path="/5470C606/5470F4EE" Ref="#PWR050"  Part="1"
 F 0 "#PWR050" H 3500 5250 30  0001 C CNN
 F 1 "GND" H 3500 5180 30  0001 C CNN
@@
 Connection ~ 7350 3950
 $Comp
-L GND #PWR051
+L GND-RESCUE-qrpamp #PWR051
 U 1 1 5470F5FC
 P 7100 4500
+AR Path="/5470F5FC" Ref="#PWR051"  Part="1"
+AR Path="/5470C606/5470F5FC" Ref="#PWR051"  Part="1"
 F 0 "#PWR051" H 7100 4500 30  0001 C CNN
 F 1 "GND" H 7100 4430 30  0001 C CNN
@@
 $EndComp
 $Comp
-L GND #PWR052
+L GND-RESCUE-qrpamp #PWR052
 U 1 1 5470F610
 P 7100 5600
+AR Path="/5470F610" Ref="#PWR052"  Part="1"
+AR Path="/5470C606/5470F610" Ref="#PWR052"  Part="1"
 F 0 "#PWR052" H 7100 5600 30  0001 C CNN
 F 1 "GND" H 7100 5530 30  0001 C CNN
@@
 amp_in
 $Comp
-L GND #PWR053
+L GND-RESCUE-qrpamp #PWR053
 U 1 1 5470F625
 P 9300 5200
+AR Path="/5470F625" Ref="#PWR053"  Part="1"
+AR Path="/5470C606/5470F625" Ref="#PWR053"  Part="1"
 F 0 "#PWR053" H 9300 5200 30  0001 C CNN
 F 1 "GND" H 9300 5130 30  0001 C CNN
@@
 $EndComp
 $Comp
-L R R7
+L R-RESCUE-qrpamp R7
 U 1 1 5470F7C0
 P 4150 2950
+AR Path="/5470F7C0" Ref="R7"  Part="1"
+AR Path="/5470C606/5470F7C0" Ref="R7"  Part="1"
 F 0 "R7" V 4230 2950 40  0000 C CNN
 F 1 "5k" V 4157 2951 40  0000 C CNN
@@
 $EndComp
 $Comp
-L R R10
+L R-RESCUE-qrpamp R10
 U 1 1 5470F7D4
 P 5000 2950
+AR Path="/5470F7D4" Ref="R10"  Part="1"
+AR Path="/5470C606/5470F7D4" Ref="R10"  Part="1"
 F 0 "R10" V 5080 2950 40  0000 C CNN
 F 1 "5k" V 5007 2951 40  0000 C CNN
@@
 $EndComp
 $Comp
-L R R9
+L R-RESCUE-qrpamp R9
 U 1 1 5470F7FC
 P 4550 2450
+AR Path="/5470F7FC" Ref="R9"  Part="1"
+AR Path="/5470C606/5470F7FC" Ref="R9"  Part="1"
 F 0 "R9" V 4630 2450 40  0000 C CNN
 F 1 "10k" V 4557 2451 40  0000 C CNN
@@
 $EndComp
 $Comp
-L R R13
+L R-RESCUE-qrpamp R13
 U 1 1 5470F80E
 P 5400 2450
+AR Path="/5470F80E" Ref="R13"  Part="1"
+AR Path="/5470C606/5470F80E" Ref="R13"  Part="1"
 F 0 "R13" V 5480 2450 40  0000 C CNN
 F 1 "10k" V 5407 2451 40  0000 C CNN
@@
 $EndComp
 $Comp
-L GND #PWR055
+L GND-RESCUE-qrpamp #PWR055
 U 1 1 5470F84C
 P 2900 2250
+AR Path="/5470F84C" Ref="#PWR055"  Part="1"
+AR Path="/5470C606/5470F84C" Ref="#PWR055"  Part="1"
 F 0 "#PWR055" H 2900 2250 30  0001 C CNN
 F 1 "GND" H 2900 2180 30  0001 C CNN
@@
 $EndComp
 $Comp
-L C C17
+L C-RESCUE-qrpamp C17
 U 1 1 5470F9F4
 P 7550 3750
+AR Path="/5470F9F4" Ref="C17"  Part="1"
+AR Path="/5470C606/5470F9F4" Ref="C17"  Part="1"
 F 0 "C17" H 7550 3850 40  0000 L CNN
 F 1 "0.1u" H 7556 3665 40  0000 L CNN
@@
 $EndComp
 $Comp
-L GND #PWR057
+L GND-RESCUE-qrpamp #PWR057
 U 1 1 5470FA0D
 P 7750 3750
+AR Path="/5470FA0D" Ref="#PWR057"  Part="1"
+AR Path="/5470C606/5470FA0D" Ref="#PWR057"  Part="1"
 F 0 "#PWR057" H 7750 3750 30  0001 C CNN
 F 1 "GND" H 7750 3680 30  0001 C CNN
@@
 $EndComp
 $Comp
-L GND #PWR058
+L GND-RESCUE-qrpamp #PWR058
 U 1 1 5470FB98
 P 5900 4850
+AR Path="/5470FB98" Ref="#PWR058"  Part="1"
+AR Path="/5470C606/5470FB98" Ref="#PWR058"  Part="1"
 F 0 "#PWR058" H 5900 4850 30  0001 C CNN
 F 1 "GND" H 5900 4780 30  0001 C CNN
@@
 	4150 1900 4150 1600
 $Comp
-L GND #PWR059
+L GND-RESCUE-qrpamp #PWR059
 U 1 1 5596F601
 P 4150 3200
+AR Path="/5596F601" Ref="#PWR059"  Part="1"
+AR Path="/5470C606/5596F601" Ref="#PWR059"  Part="1"
 F 0 "#PWR059" H 4150 3200 30  0001 C CNN
 F 1 "GND" H 4150 3130 30  0001 C CNN
@@
 $EndComp
 $Comp
-L GND #PWR060
+L GND-RESCUE-qrpamp #PWR060
 U 1 1 5596F624
 P 5000 3200
+AR Path="/5596F624" Ref="#PWR060"  Part="1"
+AR Path="/5470C606/5596F624" Ref="#PWR060"  Part="1"
 F 0 "#PWR060" H 5000 3200 30  0001 C CNN
 F 1 "GND" H 5000 3130 30  0001 C CNN
@@
 $EndComp
 $Comp
-L R R18
+L R-RESCUE-qrpamp R18
 U 1 1 55970003
 P 2650 1900
+AR Path="/55970003" Ref="R18"  Part="1"
+AR Path="/5470C606/55970003" Ref="R18"  Part="1"
 F 0 "R18" V 2730 1900 40  0000 C CNN
 F 1 "150" V 2657 1901 40  0000 C CNN
