File: mcu.sch (KiCad schematic (older format))
At the start: 9 parts

Commit message: Annotated all schematics
- Added more caps to power supply
- Decided on power supply fuse part
- Changed 1n5711 SWR caps to BAT62
- Decided on MMBF170 for amp bias switch
Parts:
- gave numbers to parts that had none: 9
Changed lines of the file:
@@
 $EndDescr
 $Comp
-L CONN_6 P?
+L CONN_6 P3
 U 1 1 5472469B
 P 3700 1550
-F 0 "P?" V 3650 1550 60  0000 C CNN
+F 0 "P3" V 3650 1550 60  0000 C CNN
 F 1 "SWD" V 3750 1550 60  0000 C CNN
 F 2 "" H 3700 1550 60  0000 C CNN
@@
 SWO
 $Comp
-L CP1 C?
+L CP1 C30
 U 1 1 54725387
 P 5350 1500
-F 0 "C?" H 5400 1600 50  0000 L CNN
+F 0 "C30" H 5400 1600 50  0000 L CNN
 F 1 "4.7u" H 5400 1400 50  0000 L CNN
 F 2 "" H 5350 1500 60  0000 C CNN
@@
 $EndComp
 $Comp
-L GND #PWR?
+L GND #PWR79
 U 1 1 547253A0
 P 5150 1500
-F 0 "#PWR?" H 5150 1500 30  0001 C CNN
+F 0 "#PWR79" H 5150 1500 30  0001 C CNN
 F 1 "GND" H 5150 1430 30  0001 C CNN
 F 2 "" H 5150 1500 60  0000 C CNN
@@
 $EndComp
 $Comp
-L CP1 C?
+L CP1 C31
 U 1 1 547253BF
 P 6200 1600
-F 0 "C?" H 6250 1700 50  0000 L CNN
+F 0 "C31" H 6250 1700 50  0000 L CNN
 F 1 "4.7u" H 6250 1500 50  0000 L CNN
 F 2 "" H 6200 1600 60  0000 C CNN
@@
 $EndComp
 $Comp
-L C C?
+L C C32
 U 1 1 547253CC
 P 6450 1600
-F 0 "C?" H 6450 1700 40  0000 L CNN
+F 0 "C32" H 6450 1700 40  0000 L CNN
 F 1 ".1u" H 6456 1515 40  0000 L CNN
 F 2 "" H 6488 1450 30  0000 C CNN
@@
 $EndComp
 $Comp
-L C C?
+L C C33
 U 1 1 547253DE
 P 6650 1600
-F 0 "C?" H 6650 1700 40  0000 L CNN
+F 0 "C33" H 6650 1700 40  0000 L CNN
 F 1 ".1u" H 6656 1515 40  0000 L CNN
 F 2 "" H 6688 1450 30  0000 C CNN
@@
 $EndComp
 $Comp
-L C C?
+L C C34
 U 1 1 547253E9
 P 6850 1600
-F 0 "C?" H 6850 1700 40  0000 L CNN
+F 0 "C34" H 6850 1700 40  0000 L CNN
 F 1 ".1u" H 6856 1515 40  0000 L CNN
 F 2 "" H 6888 1450 30  0000 C CNN
@@
 $EndComp
 $Comp
-L GND #PWR?
+L GND #PWR81
 U 1 1 54725403
 P 6850 1800
-F 0 "#PWR?" H 6850 1800 30  0001 C CNN
+F 0 "#PWR81" H 6850 1800 30  0001 C CNN
 F 1 "GND" H 6850 1730 30  0001 C CNN
 F 2 "" H 6850 1800 60  0000 C CNN
@@
 $EndComp
 $Comp
-L GND #PWR?
+L GND #PWR78
 U 1 1 5472548C
 P 4900 5350
-F 0 "#PWR?" H 4900 5350 30  0001 C CNN
+F 0 "#PWR78" H 4900 5350 30  0001 C CNN
 F 1 "GND" H 4900 5280 30  0001 C CNN
 F 2 "" H 4900 5350 60  0000 C CNN
@@
 $EndComp
 $Comp
-L GND #PWR?
+L GND #PWR75
 U 1 1 547254B6
 P 4200 1850
-F 0 "#PWR?" H 4200 1850 30  0001 C CNN
+F 0 "#PWR75" H 4200 1850 30  0001 C CNN
 F 1 "GND" H 4200 1780 30  0001 C CNN
 F 2 "" H 4200 1850 60  0000 C CNN
@@
 $EndComp
 $Comp
-L +3.3V #PWR?
+L +3.3V #PWR80
 U 1 1 547254E1
 P 5950 1400
-F 0 "#PWR?" H 5950 1360 30  0001 C CNN
+F 0 "#PWR80" H 5950 1360 30  0001 C CNN
 F 1 "+3.3V" H 5950 1510 30  0000 C CNN
 F 2 "" H 5950 1400 60  0000 C CNN
@@
 $EndComp
 $Comp
-L +3.3V #PWR?
+L +3.3V #PWR74
 U 1 1 547254F3
 P 4050 1800
-F 0 "#PWR?" H 4050 1760 30  0001 C CNN
+F 0 "#PWR74" H 4050 1760 30  0001 C CNN
 F 1 "+3.3V" H 4050 1910 30  0000 C CNN
 F 2 "" H 4050 1800 60  0000 C CNN
@@
 $EndComp
 $Comp
-L +3.3V #PWR?
+L +3.3V #PWR72
 U 1 1 547256B9
 P 800 800
-F 0 "#PWR?" H 800 760 30  0001 C CNN
+F 0 "#PWR72" H 800 760 30  0001 C CNN
 F 1 "+3.3V" H 800 910 30  0000 C CNN
 F 2 "" H 800 800 60  0000 C CNN
@@
 $EndComp
 $Comp
-L GND #PWR?
+L GND #PWR73
 U 1 1 547256C4
 P 800 900
-F 0 "#PWR?" H 800 900 30  0001 C CNN
+F 0 "#PWR73" H 800 900 30  0001 C CNN
 F 1 "GND" H 800 830 30  0001 C CNN
 F 2 "" H 800 900 60  0000 C CNN
@@
 mcu_gnd
 $Comp
-L +3.3V #PWR?
+L +3.3V #PWR76
 U 1 1 54725A58
 P 4200 3750
-F 0 "#PWR?" H 4200 3710 30  0001 C CNN
+F 0 "#PWR76" H 4200 3710 30  0001 C CNN
 F 1 "+3.3V" H 4200 3860 30  0000 C CNN
 F 2 "" H 4200 3750 60  0000 C CNN
@@
 $EndComp
 $Comp
-L GND #PWR?
+L GND #PWR77
 U 1 1 54725A7F
 P 4200 4100
-F 0 "#PWR?" H 4200 4100 30  0001 C CNN
+F 0 "#PWR77" H 4200 4100 30  0001 C CNN
 F 1 "GND" H 4200 4030 30  0001 C CNN
 F 2 "" H 4200 4100 60  0000 C CNN
@@
 $EndComp
 $Comp
-L LCD-2x16 U?
+L LCD-2x16 U3
 U 1 1 54725AD2
 P 4150 3800
-F 0 "U?" H 3675 4025 60  0000 C CNN
+F 0 "U3" H 3675 4025 60  0000 C CNN
 F 1 "LCD-2x16" H 3850 3925 60  0000 C CNN
 F 2 "" H 4150 3800 60  0000 C CNN
@@
 $EndComp
 $Comp
-L Thumb-Joystick U?
+L Thumb-Joystick U5
 U 1 1 54725DA4
 P 7950 3900
-F 0 "U?" H 7100 4125 60  0000 C CNN
+F 0 "U5" H 7100 4125 60  0000 C CNN
 F 1 "Thumb-Joystick" H 7400 4050 60  0000 C CNN
 F 2 "" H 7950 2950 60  0000 C CNN
@@
 $EndComp
 $Comp
-L STM32F401xB/C-LQFP U?
+L STM32F401xB/C-LQFP U4
 U 1 1 54725F07
 P 5200 2000
-F 0 "U?" H 6225 2100 60  0000 C CNN
+F 0 "U4" H 6225 2100 60  0000 C CNN
 F 1 "STM32F401xB/C-LQFP" H 6700 2025 60  0000 C CNN
 F 2 "" H 7175 3100 60  0000 C CNN
@@
 	7750 4200 6450 4200
 $Comp
-L GND #PWR?
+L GND #PWR86
 U 1 1 54725FF5
 P 7950 4650
-F 0 "#PWR?" H 7950 4650 30  0001 C CNN
+F 0 "#PWR86" H 7950 4650 30  0001 C CNN
 F 1 "GND" H 7950 4580 30  0001 C CNN
 F 2 "" H 7950 4650 60  0000 C CNN
@@
 $EndComp
 $Comp
-L GND #PWR?
+L GND #PWR83
 U 1 1 54726000
 P 7900 4400
-F 0 "#PWR?" H 7900 4400 30  0001 C CNN
+F 0 "#PWR83" H 7900 4400 30  0001 C CNN
 F 1 "GND" H 7900 4330 30  0001 C CNN
 F 2 "" H 7900 4400 60  0000 C CNN
@@
 $EndComp
 $Comp
-L GND #PWR?
+L GND #PWR82
 U 1 1 5472600B
 P 7900 4100
-F 0 "#PWR?" H 7900 4100 30  0001 C CNN
+F 0 "#PWR82" H 7900 4100 30  0001 C CNN
 F 1 "GND" H 7900 4030 30  0001 C CNN
 F 2 "" H 7900 4100 60  0000 C CNN
@@
 	7950 4600 7950 4650
 $Comp
-L +3.3V #PWR?
+L +3.3V #PWR84
 U 1 1 5472608E
 P 7950 3900
-F 0 "#PWR?" H 7950 3860 30  0001 C CNN
+F 0 "#PWR84" H 7950 3860 30  0001 C CNN
 F 1 "+3.3V" H 7950 4010 30  0000 C CNN
 F 2 "" H 7950 3900 60  0000 C CNN
@@
 $EndComp
 $Comp
-L +3.3V #PWR?
+L +3.3V #PWR85
 U 1 1 54726099
 P 7950 4200
-F 0 "#PWR?" H 7950 4160 30  0001 C CNN
+F 0 "#PWR85" H 7950 4160 30  0001 C CNN
 F 1 "+3.3V" H 7950 4310 30  0000 C CNN
 F 2 "" H 7950 4200 60  0000 C CNN

Commit message: Associate more footprints
- Removed flyback diodes from amp
- Changed BAT62 -> SD101 (BAT62 is EOL)
- Changed R and C footprints for hand-soldered versions
- Associated through-hole cap footprints
- Associated regulator footprints
Parts:
- C32, C33, C34: footprint (none) -> Capacitors_SMD:C_0805_HandSoldering
- U4: footprint (none) -> nu9j-footprints:LQFP64
Changed lines of the file:
@@
 LIBS:transformers
 LIBS:qrpamp-cache
-EELAYER 24 0
+EELAYER 25 0
 EELAYER END
 $Descr A4 11693 8268
@@
 F 0 "P3" V 3650 1550 60  0000 C CNN
 F 1 "SWD" V 3750 1550 60  0000 C CNN
-F 2 "" H 3700 1550 60  0000 C CNN
+F 2 "" H 3700 1550 60  0001 C CNN
 F 3 "" H 3700 1550 60  0000 C CNN
 	1    3700 1550
@@
 F 0 "C30" H 5400 1600 50  0000 L CNN
 F 1 "4.7u" H 5400 1400 50  0000 L CNN
-F 2 "" H 5350 1500 60  0000 C CNN
+F 2 "" H 5350 1500 60  0001 C CNN
 F 3 "" H 5350 1500 60  0000 C CNN
 	1    5350 1500
@@
 F 0 "C31" H 6250 1700 50  0000 L CNN
 F 1 "4.7u" H 6250 1500 50  0000 L CNN
-F 2 "" H 6200 1600 60  0000 C CNN
+F 2 "" H 6200 1600 60  0001 C CNN
 F 3 "" H 6200 1600 60  0000 C CNN
 	1    6200 1600
@@
 F 0 "C32" H 6450 1700 40  0000 L CNN
 F 1 ".1u" H 6456 1515 40  0000 L CNN
-F 2 "" H 6488 1450 30  0000 C CNN
+F 2 "Capacitors_SMD:C_0805_HandSoldering" H 6488 1450 30  0001 C CNN
 F 3 "" H 6450 1600 60  0000 C CNN
 	1    6450 1600
@@
 F 0 "C33" H 6650 1700 40  0000 L CNN
 F 1 ".1u" H 6656 1515 40  0000 L CNN
-F 2 "" H 6688 1450 30  0000 C CNN
+F 2 "Capacitors_SMD:C_0805_HandSoldering" H 6688 1450 30  0001 C CNN
 F 3 "" H 6650 1600 60  0000 C CNN
 	1    6650 1600
@@
 F 0 "C34" H 6850 1700 40  0000 L CNN
 F 1 ".1u" H 6856 1515 40  0000 L CNN
-F 2 "" H 6888 1450 30  0000 C CNN
+F 2 "Capacitors_SMD:C_0805_HandSoldering" H 6888 1450 30  0001 C CNN
 F 3 "" H 6850 1600 60  0000 C CNN
 	1    6850 1600
@@
 F 0 "U3" H 3675 4025 60  0000 C CNN
 F 1 "LCD-2x16" H 3850 3925 60  0000 C CNN
-F 2 "" H 4150 3800 60  0000 C CNN
+F 2 "" H 4150 3800 60  0001 C CNN
 F 3 "" H 4150 3800 60  0000 C CNN
 	1    4150 3800
@@
 F 0 "U5" H 7100 4125 60  0000 C CNN
 F 1 "Thumb-Joystick" H 7400 4050 60  0000 C CNN
-F 2 "" H 7950 2950 60  0000 C CNN
+F 2 "" H 7950 2950 60  0001 C CNN
 F 3 "" H 7950 2950 60  0000 C CNN
 	1    7950 3900
@@
 F 0 "U4" H 6225 2100 60  0000 C CNN
 F 1 "STM32F401xB/C-LQFP" H 6700 2025 60  0000 C CNN
-F 2 "" H 7175 3100 60  0000 C CNN
+F 2 "nu9j-footprints:LQFP64" H 7175 3100 60  0001 C CNN
 F 3 "" H 7175 3100 60  0000 C CNN
 	1    5200 2000

Commit message: Finished band filters schematic
- Associated last of the capacitors with footprints
- Associated inductors
Parts:
- C30, C31: footprint (none) -> Capacitors_ThroughHole:Capacitor5x11RM2.5
Changed lines of the file:
@@
 F 0 "C30" H 5400 1600 50  0000 L CNN
 F 1 "4.7u" H 5400 1400 50  0000 L CNN
-F 2 "" H 5350 1500 60  0001 C CNN
+F 2 "Capacitors_ThroughHole:Capacitor5x11RM2.5" H 5350 1500 60  0001 C CNN
 F 3 "" H 5350 1500 60  0000 C CNN
 	1    5350 1500
@@
 $EndComp
 $Comp
-L GND #PWR79
+L GND #PWR072
 U 1 1 547253A0
 P 5150 1500
-F 0 "#PWR79" H 5150 1500 30  0001 C CNN
+F 0 "#PWR072" H 5150 1500 30  0001 C CNN
 F 1 "GND" H 5150 1430 30  0001 C CNN
 F 2 "" H 5150 1500 60  0000 C CNN
@@
 F 0 "C31" H 6250 1700 50  0000 L CNN
 F 1 "4.7u" H 6250 1500 50  0000 L CNN
-F 2 "" H 6200 1600 60  0001 C CNN
+F 2 "Capacitors_ThroughHole:Capacitor5x11RM2.5" H 6200 1600 60  0001 C CNN
 F 3 "" H 6200 1600 60  0000 C CNN
 	1    6200 1600
@@
 $EndComp
 $Comp
-L GND #PWR81
+L GND #PWR073
 U 1 1 54725403
 P 6850 1800
-F 0 "#PWR81" H 6850 1800 30  0001 C CNN
+F 0 "#PWR073" H 6850 1800 30  0001 C CNN
 F 1 "GND" H 6850 1730 30  0001 C CNN
 F 2 "" H 6850 1800 60  0000 C CNN
@@
 $EndComp
 $Comp
-L GND #PWR78
+L GND #PWR074
 U 1 1 5472548C
 P 4900 5350
-F 0 "#PWR78" H 4900 5350 30  0001 C CNN
+F 0 "#PWR074" H 4900 5350 30  0001 C CNN
 F 1 "GND" H 4900 5280 30  0001 C CNN
 F 2 "" H 4900 5350 60  0000 C CNN
@@
 $EndComp
 $Comp
-L GND #PWR75
+L GND #PWR075
 U 1 1 547254B6
 P 4200 1850
-F 0 "#PWR75" H 4200 1850 30  0001 C CNN
+F 0 "#PWR075" H 4200 1850 30  0001 C CNN
 F 1 "GND" H 4200 1780 30  0001 C CNN
 F 2 "" H 4200 1850 60  0000 C CNN
@@
 $EndComp
 $Comp
-L +3.3V #PWR80
+L +3.3V #PWR076
 U 1 1 547254E1
 P 5950 1400
-F 0 "#PWR80" H 5950 1360 30  0001 C CNN
+F 0 "#PWR076" H 5950 1360 30  0001 C CNN
 F 1 "+3.3V" H 5950 1510 30  0000 C CNN
 F 2 "" H 5950 1400 60  0000 C CNN
@@
 $EndComp
 $Comp
-L +3.3V #PWR74
+L +3.3V #PWR077
 U 1 1 547254F3
 P 4050 1800
-F 0 "#PWR74" H 4050 1760 30  0001 C CNN
+F 0 "#PWR077" H 4050 1760 30  0001 C CNN
 F 1 "+3.3V" H 4050 1910 30  0000 C CNN
 F 2 "" H 4050 1800 60  0000 C CNN
@@
 $EndComp
 $Comp
-L +3.3V #PWR72
+L +3.3V #PWR078
 U 1 1 547256B9
 P 800 800
-F 0 "#PWR72" H 800 760 30  0001 C CNN
+F 0 "#PWR078" H 800 760 30  0001 C CNN
 F 1 "+3.3V" H 800 910 30  0000 C CNN
 F 2 "" H 800 800 60  0000 C CNN
@@
 $EndComp
 $Comp
-L GND #PWR73
+L GND #PWR079
 U 1 1 547256C4
 P 800 900
-F 0 "#PWR73" H 800 900 30  0001 C CNN
+F 0 "#PWR079" H 800 900 30  0001 C CNN
 F 1 "GND" H 800 830 30  0001 C CNN
 F 2 "" H 800 900 60  0000 C CNN
@@
 mcu_gnd
 $Comp
-L +3.3V #PWR76
+L +3.3V #PWR080
 U 1 1 54725A58
 P 4200 3750
-F 0 "#PWR76" H 4200 3710 30  0001 C CNN
+F 0 "#PWR080" H 4200 3710 30  0001 C CNN
 F 1 "+3.3V" H 4200 3860 30  0000 C CNN
 F 2 "" H 4200 3750 60  0000 C CNN
@@
 $EndComp
 $Comp
-L GND #PWR77
+L GND #PWR081
 U 1 1 54725A7F
 P 4200 4100
-F 0 "#PWR77" H 4200 4100 30  0001 C CNN
+F 0 "#PWR081" H 4200 4100 30  0001 C CNN
 F 1 "GND" H 4200 4030 30  0001 C CNN
 F 2 "" H 4200 4100 60  0000 C CNN
@@
 	7750 4200 6450 4200
 $Comp
-L GND #PWR86
+L GND #PWR082
 U 1 1 54725FF5
 P 7950 4650
-F 0 "#PWR86" H 7950 4650 30  0001 C CNN
+F 0 "#PWR082" H 7950 4650 30  0001 C CNN
 F 1 "GND" H 7950 4580 30  0001 C CNN
 F 2 "" H 7950 4650 60  0000 C CNN
@@
 $EndComp
 $Comp
-L GND #PWR83
+L GND #PWR083
 U 1 1 54726000
 P 7900 4400
-F 0 "#PWR83" H 7900 4400 30  0001 C CNN
+F 0 "#PWR083" H 7900 4400 30  0001 C CNN
 F 1 "GND" H 7900 4330 30  0001 C CNN
 F 2 "" H 7900 4400 60  0000 C CNN
@@
 $EndComp
 $Comp
-L GND #PWR82
+L GND #PWR084
 U 1 1 5472600B
 P 7900 4100
-F 0 "#PWR82" H 7900 4100 30  0001 C CNN
+F 0 "#PWR084" H 7900 4100 30  0001 C CNN
 F 1 "GND" H 7900 4030 30  0001 C CNN
 F 2 "" H 7900 4100 60  0000 C CNN
@@
 	7950 4600 7950 4650
 $Comp
-L +3.3V #PWR84
+L +3.3V #PWR085
 U 1 1 5472608E
 P 7950 3900
-F 0 "#PWR84" H 7950 3860 30  0001 C CNN
+F 0 "#PWR085" H 7950 3860 30  0001 C CNN
 F 1 "+3.3V" H 7950 4010 30  0000 C CNN
 F 2 "" H 7950 3900 60  0000 C CNN
@@
 $EndComp
 $Comp
-L +3.3V #PWR85
+L +3.3V #PWR086
 U 1 1 54726099
 P 7950 4200
-F 0 "#PWR85" H 7950 4160 30  0001 C CNN
+F 0 "#PWR086" H 7950 4160 30  0001 C CNN
 F 1 "+3.3V" H 7950 4310 30  0000 C CNN
 F 2 "" H 7950 4200 60  0000 C CNN

Commit message: Finished associating relays
Parts:
- P3: footprint (none) -> Pin_Headers:Pin_Header_Straight_1x06
Changed lines of the file:
@@
 LIBS:mcus
 LIBS:transformers
+LIBS:relays
 LIBS:qrpamp-cache
 EELAYER 25 0
@@
 F 0 "P3" V 3650 1550 60  0000 C CNN
 F 1 "SWD" V 3750 1550 60  0000 C CNN
-F 2 "" H 3700 1550 60  0001 C CNN
+F 2 "Pin_Headers:Pin_Header_Straight_1x06" H 3700 1550 60  0001 C CNN
 F 3 "" H 3700 1550 60  0000 C CNN
 	1    3700 1550
@@
 $EndComp
 $Comp
-L GND #PWR072
+L GND #PWR78
 U 1 1 547253A0
 P 5150 1500
-F 0 "#PWR072" H 5150 1500 30  0001 C CNN
+F 0 "#PWR78" H 5150 1500 30  0001 C CNN
 F 1 "GND" H 5150 1430 30  0001 C CNN
 F 2 "" H 5150 1500 60  0000 C CNN
@@
 $EndComp
 $Comp
-L GND #PWR073
+L GND #PWR80
 U 1 1 54725403
 P 6850 1800
-F 0 "#PWR073" H 6850 1800 30  0001 C CNN
+F 0 "#PWR80" H 6850 1800 30  0001 C CNN
 F 1 "GND" H 6850 1730 30  0001 C CNN
 F 2 "" H 6850 1800 60  0000 C CNN
@@
 $EndComp
 $Comp
-L GND #PWR074
+L GND #PWR77
 U 1 1 5472548C
 P 4900 5350
-F 0 "#PWR074" H 4900 5350 30  0001 C CNN
+F 0 "#PWR77" H 4900 5350 30  0001 C CNN
 F 1 "GND" H 4900 5280 30  0001 C CNN
 F 2 "" H 4900 5350 60  0000 C CNN
@@
 $EndComp
 $Comp
-L GND #PWR075
+L GND #PWR74
 U 1 1 547254B6
 P 4200 1850
-F 0 "#PWR075" H 4200 1850 30  0001 C CNN
+F 0 "#PWR74" H 4200 1850 30  0001 C CNN
 F 1 "GND" H 4200 1780 30  0001 C CNN
 F 2 "" H 4200 1850 60  0000 C CNN
@@
 $EndComp
 $Comp
-L +3.3V #PWR076
+L +3.3V #PWR79
 U 1 1 547254E1
 P 5950 1400
-F 0 "#PWR076" H 5950 1360 30  0001 C CNN
+F 0 "#PWR79" H 5950 1360 30  0001 C CNN
 F 1 "+3.3V" H 5950 1510 30  0000 C CNN
 F 2 "" H 5950 1400 60  0000 C CNN
@@
 $EndComp
 $Comp
-L +3.3V #PWR077
+L +3.3V #PWR73
 U 1 1 547254F3
 P 4050 1800
-F 0 "#PWR077" H 4050 1760 30  0001 C CNN
+F 0 "#PWR73" H 4050 1760 30  0001 C CNN
 F 1 "+3.3V" H 4050 1910 30  0000 C CNN
 F 2 "" H 4050 1800 60  0000 C CNN
@@
 $EndComp
 $Comp
-L +3.3V #PWR078
+L +3.3V #PWR71
 U 1 1 547256B9
 P 800 800
-F 0 "#PWR078" H 800 760 30  0001 C CNN
+F 0 "#PWR71" H 800 760 30  0001 C CNN
 F 1 "+3.3V" H 800 910 30  0000 C CNN
 F 2 "" H 800 800 60  0000 C CNN
@@
 $EndComp
 $Comp
-L GND #PWR079
+L GND #PWR72
 U 1 1 547256C4
 P 800 900
-F 0 "#PWR079" H 800 900 30  0001 C CNN
+F 0 "#PWR72" H 800 900 30  0001 C CNN
 F 1 "GND" H 800 830 30  0001 C CNN
 F 2 "" H 800 900 60  0000 C CNN
@@
 mcu_gnd
 $Comp
-L +3.3V #PWR080
+L +3.3V #PWR75
 U 1 1 54725A58
 P 4200 3750
-F 0 "#PWR080" H 4200 3710 30  0001 C CNN
+F 0 "#PWR75" H 4200 3710 30  0001 C CNN
 F 1 "+3.3V" H 4200 3860 30  0000 C CNN
 F 2 "" H 4200 3750 60  0000 C CNN
@@
 $EndComp
 $Comp
-L GND #PWR081
+L GND #PWR76
 U 1 1 54725A7F
 P 4200 4100
-F 0 "#PWR081" H 4200 4100 30  0001 C CNN
+F 0 "#PWR76" H 4200 4100 30  0001 C CNN
 F 1 "GND" H 4200 4030 30  0001 C CNN
 F 2 "" H 4200 4100 60  0000 C CNN
@@
 	7750 4200 6450 4200
 $Comp
-L GND #PWR082
+L GND #PWR85
 U 1 1 54725FF5
 P 7950 4650
-F 0 "#PWR082" H 7950 4650 30  0001 C CNN
+F 0 "#PWR85" H 7950 4650 30  0001 C CNN
 F 1 "GND" H 7950 4580 30  0001 C CNN
 F 2 "" H 7950 4650 60  0000 C CNN
@@
 $EndComp
 $Comp
-L GND #PWR083
+L GND #PWR82
 U 1 1 54726000
 P 7900 4400
-F 0 "#PWR083" H 7900 4400 30  0001 C CNN
+F 0 "#PWR82" H 7900 4400 30  0001 C CNN
 F 1 "GND" H 7900 4330 30  0001 C CNN
 F 2 "" H 7900 4400 60  0000 C CNN
@@
 $EndComp
 $Comp
-L GND #PWR084
+L GND #PWR81
 U 1 1 5472600B
 P 7900 4100
-F 0 "#PWR084" H 7900 4100 30  0001 C CNN
+F 0 "#PWR81" H 7900 4100 30  0001 C CNN
 F 1 "GND" H 7900 4030 30  0001 C CNN
 F 2 "" H 7900 4100 60  0000 C CNN
@@
 	7950 4600 7950 4650
 $Comp
-L +3.3V #PWR085
+L +3.3V #PWR83
 U 1 1 5472608E
 P 7950 3900
-F 0 "#PWR085" H 7950 3860 30  0001 C CNN
+F 0 "#PWR83" H 7950 3860 30  0001 C CNN
 F 1 "+3.3V" H 7950 4010 30  0000 C CNN
 F 2 "" H 7950 3900 60  0000 C CNN
@@
 $EndComp
 $Comp
-L +3.3V #PWR086
+L +3.3V #PWR84
 U 1 1 54726099
 P 7950 4200
-F 0 "#PWR086" H 7950 4160 30  0001 C CNN
+F 0 "#PWR84" H 7950 4160 30  0001 C CNN
 F 1 "+3.3V" H 7950 4310 30  0000 C CNN
 F 2 "" H 7950 4200 60  0000 C CNN

Commit message: Everything associated except joystick
Parts:
- U3: footprint (none) -> Pin_Headers:Pin_Header_Straight_1x03
Changed lines of the file:
@@
 $EndComp
 $Comp
-L GND #PWR78
+L GND #PWR071
 U 1 1 547253A0
 P 5150 1500
-F 0 "#PWR78" H 5150 1500 30  0001 C CNN
+F 0 "#PWR071" H 5150 1500 30  0001 C CNN
 F 1 "GND" H 5150 1430 30  0001 C CNN
 F 2 "" H 5150 1500 60  0000 C CNN
@@
 $EndComp
 $Comp
-L GND #PWR80
+L GND #PWR072
 U 1 1 54725403
 P 6850 1800
-F 0 "#PWR80" H 6850 1800 30  0001 C CNN
+F 0 "#PWR072" H 6850 1800 30  0001 C CNN
 F 1 "GND" H 6850 1730 30  0001 C CNN
 F 2 "" H 6850 1800 60  0000 C CNN
@@
 $EndComp
 $Comp
-L GND #PWR77
+L GND #PWR073
 U 1 1 5472548C
 P 4900 5350
-F 0 "#PWR77" H 4900 5350 30  0001 C CNN
+F 0 "#PWR073" H 4900 5350 30  0001 C CNN
 F 1 "GND" H 4900 5280 30  0001 C CNN
 F 2 "" H 4900 5350 60  0000 C CNN
@@
 $EndComp
 $Comp
-L GND #PWR74
+L GND #PWR074
 U 1 1 547254B6
 P 4200 1850
-F 0 "#PWR74" H 4200 1850 30  0001 C CNN
+F 0 "#PWR074" H 4200 1850 30  0001 C CNN
 F 1 "GND" H 4200 1780 30  0001 C CNN
 F 2 "" H 4200 1850 60  0000 C CNN
@@
 $EndComp
 $Comp
-L +3.3V #PWR79
+L +3.3V #PWR075
 U 1 1 547254E1
 P 5950 1400
-F 0 "#PWR79" H 5950 1360 30  0001 C CNN
+F 0 "#PWR075" H 5950 1360 30  0001 C CNN
 F 1 "+3.3V" H 5950 1510 30  0000 C CNN
 F 2 "" H 5950 1400 60  0000 C CNN
@@
 $EndComp
 $Comp
-L +3.3V #PWR73
+L +3.3V #PWR076
 U 1 1 547254F3
 P 4050 1800
-F 0 "#PWR73" H 4050 1760 30  0001 C CNN
+F 0 "#PWR076" H 4050 1760 30  0001 C CNN
 F 1 "+3.3V" H 4050 1910 30  0000 C CNN
 F 2 "" H 4050 1800 60  0000 C CNN
@@
 $EndComp
 $Comp
-L +3.3V #PWR71
+L +3.3V #PWR077
 U 1 1 547256B9
 P 800 800
-F 0 "#PWR71" H 800 760 30  0001 C CNN
+F 0 "#PWR077" H 800 760 30  0001 C CNN
 F 1 "+3.3V" H 800 910 30  0000 C CNN
 F 2 "" H 800 800 60  0000 C CNN
@@
 $EndComp
 $Comp
-L GND #PWR72
+L GND #PWR078
 U 1 1 547256C4
 P 800 900
-F 0 "#PWR72" H 800 900 30  0001 C CNN
+F 0 "#PWR078" H 800 900 30  0001 C CNN
 F 1 "GND" H 800 830 30  0001 C CNN
 F 2 "" H 800 900 60  0000 C CNN
@@
 mcu_gnd
 $Comp
-L +3.3V #PWR75
+L +3.3V #PWR079
 U 1 1 54725A58
 P 4200 3750
-F 0 "#PWR75" H 4200 3710 30  0001 C CNN
+F 0 "#PWR079" H 4200 3710 30  0001 C CNN
 F 1 "+3.3V" H 4200 3860 30  0000 C CNN
 F 2 "" H 4200 3750 60  0000 C CNN
@@
 $EndComp
 $Comp
-L GND #PWR76
+L GND #PWR080
 U 1 1 54725A7F
 P 4200 4100
-F 0 "#PWR76" H 4200 4100 30  0001 C CNN
+F 0 "#PWR080" H 4200 4100 30  0001 C CNN
 F 1 "GND" H 4200 4030 30  0001 C CNN
 F 2 "" H 4200 4100 60  0000 C CNN
@@
 F 0 "U3" H 3675 4025 60  0000 C CNN
 F 1 "LCD-2x16" H 3850 3925 60  0000 C CNN
-F 2 "" H 4150 3800 60  0001 C CNN
+F 2 "Pin_Headers:Pin_Header_Straight_1x03" H 4150 3800 60  0001 C CNN
 F 3 "" H 4150 3800 60  0000 C CNN
 	1    4150 3800
@@
 	7750 4200 6450 4200
 $Comp
-L GND #PWR85
+L GND #PWR081
 U 1 1 54725FF5
 P 7950 4650
-F 0 "#PWR85" H 7950 4650 30  0001 C CNN
+F 0 "#PWR081" H 7950 4650 30  0001 C CNN
 F 1 "GND" H 7950 4580 30  0001 C CNN
 F 2 "" H 7950 4650 60  0000 C CNN
@@
 $EndComp
 $Comp
-L GND #PWR82
+L GND #PWR082
 U 1 1 54726000
 P 7900 4400
-F 0 "#PWR82" H 7900 4400 30  0001 C CNN
+F 0 "#PWR082" H 7900 4400 30  0001 C CNN
 F 1 "GND" H 7900 4330 30  0001 C CNN
 F 2 "" H 7900 4400 60  0000 C CNN
@@
 $EndComp
 $Comp
-L GND #PWR81
+L GND #PWR083
 U 1 1 5472600B
 P 7900 4100
-F 0 "#PWR81" H 7900 4100 30  0001 C CNN
+F 0 "#PWR083" H 7900 4100 30  0001 C CNN
 F 1 "GND" H 7900 4030 30  0001 C CNN
 F 2 "" H 7900 4100 60  0000 C CNN
@@
 	7950 4600 7950 4650
 $Comp
-L +3.3V #PWR83
+L +3.3V #PWR084
 U 1 1 5472608E
 P 7950 3900
-F 0 "#PWR83" H 7950 3860 30  0001 C CNN
+F 0 "#PWR084" H 7950 3860 30  0001 C CNN
 F 1 "+3.3V" H 7950 4010 30  0000 C CNN
 F 2 "" H 7950 3900 60  0000 C CNN
@@
 $EndComp
 $Comp
-L +3.3V #PWR84
+L +3.3V #PWR085
 U 1 1 54726099
 P 7950 4200
-F 0 "#PWR84" H 7950 4160 30  0001 C CNN
+F 0 "#PWR085" H 7950 4160 30  0001 C CNN
 F 1 "+3.3V" H 7950 4310 30  0000 C CNN
 F 2 "" H 7950 4200 60  0000 C CNN
