File: mcu.sch (KiCad schematic (older format))
At the start: 12 parts, among them P3 SWD, P7 Thumb-Joystick, SW1 SW_PUSH, U3 LCD-2x16, U4 STM32F401xB/C-LQFP

Commit message: Added ADC input resistors
Also reassigned the band switch pins on the 401 for better layout.
Parts:
- added R24, R25: 50k, Resistors_SMD:R_1206_HandSoldering, symbol R
Changed lines of the file:
@@
 Wire Wire Line
 	4200 4250 4200 4450
-Text HLabel 6500 2550 2    60   Output ~ 0
+Text HLabel 6500 3550 2    60   Output ~ 0
 mcu_band1
-Text HLabel 6500 2450 2    60   Output ~ 0
+Text HLabel 6500 3450 2    60   Output ~ 0
 mcu_band2
-Text HLabel 6500 2350 2    60   Output ~ 0
+Text HLabel 6500 3350 2    60   Output ~ 0
 mcu_band3
-Wire Wire Line
-	6450 2350 6500 2350
-Wire Wire Line
-	6500 2450 6450 2450
-Wire Wire Line
-	6450 2550 6500 2550
 Text HLabel 6500 5050 2    60   Input ~ 0
 mcu_rfdet
 Text HLabel 4850 3450 0    60   Input ~ 0
 mcu_ptt
-Text HLabel 6500 2950 2    60   Input ~ 0
+Text HLabel 7000 2950 2    60   Input ~ 0
 mcu_swr_fwd
-Text HLabel 6500 2850 2    60   Input ~ 0
+Text HLabel 7000 2850 2    60   Input ~ 0
 mcu_swr_ref
 Wire Wire Line
@@
 Text Label 4600 2650 0    60   ~ 0
 SWCLK
+$Comp
+L R R24
+U 1 1 548C7F6B
+P 6750 2850
+F 0 "R24" V 6830 2850 40  0000 C CNN
+F 1 "50k" V 6757 2851 40  0000 C CNN
+F 2 "Resistors_SMD:R_1206_HandSoldering" V 6680 2850 30  0001 C CNN
+F 3 "" H 6750 2850 30  0000 C CNN
+	1    6750 2850
+	0    -1   -1   0
+$EndComp
+$Comp
+L R R25
+U 1 1 548C7FD3
+P 6750 2950
+F 0 "R25" V 6830 2950 40  0000 C CNN
+F 1 "50k" V 6757 2951 40  0000 C CNN
+F 2 "Resistors_SMD:R_1206_HandSoldering" V 6680 2950 30  0001 C CNN
+F 3 "" H 6750 2950 30  0000 C CNN
+	1    6750 2950
+	0    1    1    0
+$EndComp
+Wire Wire Line
+	6450 3350 6500 3350
+Wire Wire Line
+	6500 3450 6450 3450
+Wire Wire Line
+	6450 3550 6500 3550
 $EndSCHEMATC

Commit message: Fixed issues found with test board
- Added MOSFETs to relay switch lines from MCU
- Reconnected SWR in/out to actual ADC pins
- Changed LM3940 footprint to SOT223
- Added 4th mounting hole
- Swapped joystick for nav button
- Extended pads of STM32F401 for easier soldering
Parts:
- removed P7: Thumb-Joystick, Pin_Headers:Pin_Header_Straight_1x05, symbol CONN_01X05
- added P7: TP, Measurement_Points:Measurement_Point_Round-SMD-Pad_Small, symbol CONN_01X01
- added P8: NAV_BUTTON, Pin_Headers:Pin_Header_Straight_1x06, symbol CONN_01X06
- added R26: 10k, Resistors_SMD:R_1206_HandSoldering, symbol R
Connections:
- net labels added: nav_down, nav_left, nav_right, nav_select, nav_up
- wire segments 44 -> 50
Other:
- moved on the sheet: C38, C39, R24, R25
