File: bandfilters.sch (KiCad schematic (older format))
At the start: 28 parts, among them K1 BAND3_IN, K2 BAND2_IN, K3 BAND1_IN, K4 BAND3_OUT, K5 BAND2_OUT, K6 BAND1_OUT, Q10 MMBF170, Q11 MMBF170, Q9 MMBF170

Commit message: Update project to kicad bzr 6336
I guess some parts are now outdated
Parts:
- C18, C19, C20, C21, C22, C23, C24, C25, C26, C27, C28, C29: symbol C -> C-RESCUE-qrpamp
Changed lines of the file:
@@
 EESchema Schematic File Version 2
+LIBS:qrpamp-rescue
 LIBS:power
 LIBS:device
@@
 $EndDescr
 $Comp
-L C C18
+L C-RESCUE-qrpamp C18
 U 1 1 5470D5D2
 P 5100 2350
+AR Path="/5470D5D2" Ref="C18"  Part="1"
+AR Path="/5470C620/5470D5D2" Ref="C18"  Part="1"
 F 0 "C18" H 5100 2450 40  0000 L CNN
 F 1 "150p" H 5106 2265 40  0000 L CNN
@@
 $EndComp
 $Comp
-L C C22
+L C-RESCUE-qrpamp C22
 U 1 1 5470D605
 P 5850 2350
+AR Path="/5470D605" Ref="C22"  Part="1"
+AR Path="/5470C620/5470D605" Ref="C22"  Part="1"
 F 0 "C22" H 5850 2450 40  0000 L CNN
 F 1 "270p" H 5856 2265 40  0000 L CNN
@@
 $EndComp
 $Comp
-L C C26
+L C-RESCUE-qrpamp C26
 U 1 1 5470D617
 P 6550 2350
+AR Path="/5470D617" Ref="C26"  Part="1"
+AR Path="/5470C620/5470D617" Ref="C26"  Part="1"
 F 0 "C26" H 6550 2450 40  0000 L CNN
 F 1 "150p" H 6556 2265 40  0000 L CNN
@@
 $EndComp
 $Comp
-L GND #PWR061
+L GND-RESCUE-qrpamp #PWR061
 U 1 1 5470D63D
 P 5100 2550
+AR Path="/5470D63D" Ref="#PWR061"  Part="1"
+AR Path="/5470C620/5470D63D" Ref="#PWR061"  Part="1"
 F 0 "#PWR061" H 5100 2550 30  0001 C CNN
 F 1 "GND" H 5100 2480 30  0001 C CNN
@@
 $EndComp
 $Comp
-L GND #PWR062
+L GND-RESCUE-qrpamp #PWR062
 U 1 1 5470D651
 P 5850 2550
+AR Path="/5470D651" Ref="#PWR062"  Part="1"
+AR Path="/5470C620/5470D651" Ref="#PWR062"  Part="1"
 F 0 "#PWR062" H 5850 2550 30  0001 C CNN
 F 1 "GND" H 5850 2480 30  0001 C CNN
@@
 $EndComp
 $Comp
-L GND #PWR063
+L GND-RESCUE-qrpamp #PWR063
 U 1 1 5470D665
 P 6550 2550
+AR Path="/5470D665" Ref="#PWR063"  Part="1"
+AR Path="/5470C620/5470D665" Ref="#PWR063"  Part="1"
 F 0 "#PWR063" H 6550 2550 30  0001 C CNN
 F 1 "GND" H 6550 2480 30  0001 C CNN
@@
 $EndComp
 $Comp
-L C C19
+L C-RESCUE-qrpamp C19
 U 1 1 5470D6CF
 P 5100 3650
+AR Path="/5470D6CF" Ref="C19"  Part="1"
+AR Path="/5470C620/5470D6CF" Ref="C19"  Part="1"
 F 0 "C19" H 5100 3750 40  0000 L CNN
 F 1 "330p" H 5106 3565 40  0000 L CNN
@@
 $EndComp
 $Comp
-L C C23
+L C-RESCUE-qrpamp C23
 U 1 1 5470D6E1
 P 5850 3650
+AR Path="/5470D6E1" Ref="C23"  Part="1"
+AR Path="/5470C620/5470D6E1" Ref="C23"  Part="1"
 F 0 "C23" H 5850 3750 40  0000 L CNN
 F 1 "680p" H 5856 3565 40  0000 L CNN
@@
 $EndComp
 $Comp
-L C C27
+L C-RESCUE-qrpamp C27
 U 1 1 5470D6E7
 P 6550 3650
+AR Path="/5470D6E7" Ref="C27"  Part="1"
+AR Path="/5470C620/5470D6E7" Ref="C27"  Part="1"
 F 0 "C27" H 6550 3750 40  0000 L CNN
 F 1 "330p" H 6556 3565 40  0000 L CNN
@@
 $EndComp
 $Comp
-L GND #PWR064
+L GND-RESCUE-qrpamp #PWR064
 U 1 1 5470D6F1
 P 5100 3850
+AR Path="/5470D6F1" Ref="#PWR064"  Part="1"
+AR Path="/5470C620/5470D6F1" Ref="#PWR064"  Part="1"
 F 0 "#PWR064" H 5100 3850 30  0001 C CNN
 F 1 "GND" H 5100 3780 30  0001 C CNN
@@
 $EndComp
 $Comp
-L GND #PWR065
+L GND-RESCUE-qrpamp #PWR065
 U 1 1 5470D6F7
 P 5850 3850
+AR Path="/5470D6F7" Ref="#PWR065"  Part="1"
+AR Path="/5470C620/5470D6F7" Ref="#PWR065"  Part="1"
 F 0 "#PWR065" H 5850 3850 30  0001 C CNN
 F 1 "GND" H 5850 3780 30  0001 C CNN
@@
 $EndComp
 $Comp
-L GND #PWR066
+L GND-RESCUE-qrpamp #PWR066
 U 1 1 5470D6FD
 P 6550 3850
+AR Path="/5470D6FD" Ref="#PWR066"  Part="1"
+AR Path="/5470C620/5470D6FD" Ref="#PWR066"  Part="1"
 F 0 "#PWR066" H 6550 3850 30  0001 C CNN
 F 1 "GND" H 6550 3780 30  0001 C CNN
@@
 $EndComp
 $Comp
-L C C20
+L C-RESCUE-qrpamp C20
 U 1 1 5470D703
 P 5100 4950
+AR Path="/5470D703" Ref="C20"  Part="1"
+AR Path="/5470C620/5470D703" Ref="C20"  Part="1"
 F 0 "C20" H 5100 5050 40  0000 L CNN
 F 1 "560p" H 5106 4865 40  0000 L CNN
@@
 $EndComp
 $Comp
-L C C24
+L C-RESCUE-qrpamp C24
 U 1 1 5470D715
 P 5850 4950
+AR Path="/5470D715" Ref="C24"  Part="1"
+AR Path="/5470C620/5470D715" Ref="C24"  Part="1"
 F 0 "C24" H 5850 5050 40  0000 L CNN
 F 1 "1000p" H 5856 4865 40  0000 L CNN
@@
 $EndComp
 $Comp
-L C C28
+L C-RESCUE-qrpamp C28
 U 1 1 5470D71B
 P 6550 4950
+AR Path="/5470D71B" Ref="C28"  Part="1"
+AR Path="/5470C620/5470D71B" Ref="C28"  Part="1"
 F 0 "C28" H 6550 5050 40  0000 L CNN
 F 1 "560p" H 6556 4865 40  0000 L CNN
@@
 $EndComp
 $Comp
-L GND #PWR067
+L GND-RESCUE-qrpamp #PWR067
 U 1 1 5470D725
 P 5100 5150
+AR Path="/5470D725" Ref="#PWR067"  Part="1"
+AR Path="/5470C620/5470D725" Ref="#PWR067"  Part="1"
 F 0 "#PWR067" H 5100 5150 30  0001 C CNN
 F 1 "GND" H 5100 5080 30  0001 C CNN
@@
 $EndComp
 $Comp
-L GND #PWR068
+L GND-RESCUE-qrpamp #PWR068
 U 1 1 5470D72B
 P 5850 5150
+AR Path="/5470D72B" Ref="#PWR068"  Part="1"
+AR Path="/5470C620/5470D72B" Ref="#PWR068"  Part="1"
 F 0 "#PWR068" H 5850 5150 30  0001 C CNN
 F 1 "GND" H 5850 5080 30  0001 C CNN
@@
 $EndComp
 $Comp
-L GND #PWR069
+L GND-RESCUE-qrpamp #PWR069
 U 1 1 5470D731
 P 6550 5150
+AR Path="/5470D731" Ref="#PWR069"  Part="1"
+AR Path="/5470C620/5470D731" Ref="#PWR069"  Part="1"
 F 0 "#PWR069" H 6550 5150 30  0001 C CNN
 F 1 "GND" H 6550 5080 30  0001 C CNN
@@
 $EndComp
 $Comp
-L C C21
+L C-RESCUE-qrpamp C21
 U 1 1 5470D85B
 P 5650 6000
+AR Path="/5470D85B" Ref="C21"  Part="1"
+AR Path="/5470C620/5470D85B" Ref="C21"  Part="1"
 F 0 "C21" H 5650 6100 40  0000 L CNN
 F 1 "1800p" H 5656 5915 40  0000 L CNN
@@
 $EndComp
 $Comp
-L C C25
+L C-RESCUE-qrpamp C25
 U 1 1 5470D86D
 P 5850 5800
+AR Path="/5470D86D" Ref="C25"  Part="1"
+AR Path="/5470C620/5470D86D" Ref="C25"  Part="1"
 F 0 "C25" H 5850 5900 40  0000 L CNN
 F 1 "150p" H 5856 5715 40  0000 L CNN
@@
 $EndComp
 $Comp
-L C C29
+L C-RESCUE-qrpamp C29
 U 1 1 5470D873
 P 6050 6000
+AR Path="/5470D873" Ref="C29"  Part="1"
+AR Path="/5470C620/5470D873" Ref="C29"  Part="1"
 F 0 "C29" H 6050 6100 40  0000 L CNN
 F 1 "1800p" H 6056 5915 40  0000 L CNN
@@
 $EndComp
 $Comp
-L GND #PWR070
+L GND-RESCUE-qrpamp #PWR070
 U 1 1 5470D87D
 P 5650 6200
+AR Path="/5470D87D" Ref="#PWR070"  Part="1"
+AR Path="/5470C620/5470D87D" Ref="#PWR070"  Part="1"
 F 0 "#PWR070" H 5650 6200 30  0001 C CNN
 F 1 "GND" H 5650 6130 30  0001 C CNN
@@
 $EndComp
 $Comp
-L GND #PWR071
+L GND-RESCUE-qrpamp #PWR071
 U 1 1 5470D889
 P 6050 6200
+AR Path="/5470D889" Ref="#PWR071"  Part="1"
+AR Path="/5470C620/5470D889" Ref="#PWR071"  Part="1"
 F 0 "#PWR071" H 6050 6200 30  0001 C CNN
 F 1 "GND" H 6050 6130 30  0001 C CNN
@@
 $EndComp
 $Comp
-L GND #PWR079
+L GND-RESCUE-qrpamp #PWR079
 U 1 1 5470E69D
 P 10200 900
+AR Path="/5470E69D" Ref="#PWR079"  Part="1"
+AR Path="/5470C620/5470E69D" Ref="#PWR079"  Part="1"
 F 0 "#PWR079" H 10200 900 30  0001 C CNN
 F 1 "GND" H 10200 830 30  0001 C CNN
@@
 $EndComp
 $Comp
-L GND #PWR080
+L GND-RESCUE-qrpamp #PWR080
 U 1 1 54C463F8
 P 10300 3900
+AR Path="/54C463F8" Ref="#PWR080"  Part="1"
+AR Path="/5470C620/54C463F8" Ref="#PWR080"  Part="1"
 F 0 "#PWR080" H 10300 3900 30  0001 C CNN
 F 1 "GND" H 10300 3830 30  0001 C CNN
@@
 $EndComp
 $Comp
-L GND #PWR081
+L GND-RESCUE-qrpamp #PWR081
 U 1 1 54C464EC
 P 10300 4450
+AR Path="/54C464EC" Ref="#PWR081"  Part="1"
+AR Path="/5470C620/54C464EC" Ref="#PWR081"  Part="1"
 F 0 "#PWR081" H 10300 4450 30  0001 C CNN
 F 1 "GND" H 10300 4380 30  0001 C CNN
@@
 $EndComp
 $Comp
-L GND #PWR082
+L GND-RESCUE-qrpamp #PWR082
 U 1 1 54C46558
 P 10300 5000
+AR Path="/54C46558" Ref="#PWR082"  Part="1"
+AR Path="/5470C620/54C46558" Ref="#PWR082"  Part="1"
 F 0 "#PWR082" H 10300 5000 30  0001 C CNN
 F 1 "GND" H 10300 4930 30  0001 C CNN
