File: powersupply.sch (KiCad schematic (older format))
At the start: 24 parts, among them P1 PWR, P2 PWR_SW, U1 LM7805, U2 LM3940

Commit message: Update project to kicad bzr 6336
I guess some parts are now outdated
Parts:
- C10, C12, C13, C14, C3, C9: symbol C -> C-RESCUE-qrpamp
- C11, C32, C4, C40, C41, C42, C43, C5, C6, C7, C8: symbol CP1 -> CP1-RESCUE-qrpamp
