File: rfdet.sch (KiCad schematic (older format))
At the start: 8 parts, among them Q1 MMBT6427

Commit message: Update project to kicad bzr 6336
I guess some parts are now outdated
Parts:
- C1, C2: symbol C -> C-RESCUE-qrpamp
- R1, R2, R3, R4: symbol R -> R-RESCUE-qrpamp
Changed lines of the file:
@@
 EESchema Schematic File Version 2
+LIBS:qrpamp-rescue
 LIBS:power
 LIBS:device
@@
 $EndDescr
 $Comp
-L C C1
+L C-RESCUE-qrpamp C1
 U 1 1 5470CFC5
 P 4300 3700
+AR Path="/5470CFC5" Ref="C1"  Part="1"
+AR Path="/5470C525/5470CFC5" Ref="C1"  Part="1"
 F 0 "C1" H 4300 3800 40  0000 L CNN
 F 1 ".1u" H 4306 3615 40  0000 L CNN
@@
 $EndComp
 $Comp
-L R R4
+L R-RESCUE-qrpamp R4
 U 1 1 5470D001
 P 6300 3700
+AR Path="/5470D001" Ref="R4"  Part="1"
+AR Path="/5470C525/5470D001" Ref="R4"  Part="1"
 F 0 "R4" V 6380 3700 40  0000 C CNN
 F 1 "10k" V 6307 3701 40  0000 C CNN
@@
 $EndComp
 $Comp
-L R R1
+L R-RESCUE-qrpamp R1
 U 1 1 5470D02C
 P 4600 3950
+AR Path="/5470D02C" Ref="R1"  Part="1"
+AR Path="/5470C525/5470D02C" Ref="R1"  Part="1"
 F 0 "R1" V 4680 3950 40  0000 C CNN
 F 1 "10k" V 4607 3951 40  0000 C CNN
@@
 $EndComp
 $Comp
-L GND #PWR017
+L GND-RESCUE-qrpamp #PWR017
 U 1 1 5470D04B
 P 5700 4300
+AR Path="/5470D04B" Ref="#PWR017"  Part="1"
+AR Path="/5470C525/5470D04B" Ref="#PWR017"  Part="1"
 F 0 "#PWR017" H 5700 4300 30  0001 C CNN
 F 1 "GND" H 5700 4230 30  0001 C CNN
@@
 $EndComp
 $Comp
-L GND #PWR018
+L GND-RESCUE-qrpamp #PWR018
 U 1 1 5470D056
 P 4600 4300
+AR Path="/5470D056" Ref="#PWR018"  Part="1"
+AR Path="/5470C525/5470D056" Ref="#PWR018"  Part="1"
 F 0 "#PWR018" H 4600 4300 30  0001 C CNN
 F 1 "GND" H 4600 4230 30  0001 C CNN
@@
 	6550 3700 6700 3700
 $Comp
-L GND #PWR019
+L GND-RESCUE-qrpamp #PWR019
 U 1 1 5470D254
 P 7200 4300
+AR Path="/5470D254" Ref="#PWR019"  Part="1"
+AR Path="/5470C525/5470D254" Ref="#PWR019"  Part="1"
 F 0 "#PWR019" H 7200 4300 30  0001 C CNN
 F 1 "GND" H 7200 4230 30  0001 C CNN
@@
 rfdet_gnd
 $Comp
-L R R3
+L R-RESCUE-qrpamp R3
 U 1 1 5477B801
 P 6050 3950
+AR Path="/5477B801" Ref="R3"  Part="1"
+AR Path="/5470C525/5477B801" Ref="R3"  Part="1"
 F 0 "R3" V 6130 3950 40  0000 C CNN
 F 1 "6.8k" V 6057 3951 40  0000 C CNN
@@
 $EndComp
 $Comp
-L GND #PWR020
+L GND-RESCUE-qrpamp #PWR020
 U 1 1 5477B80C
 P 6050 4300
+AR Path="/5477B80C" Ref="#PWR020"  Part="1"
+AR Path="/5470C525/5477B80C" Ref="#PWR020"  Part="1"
 F 0 "#PWR020" H 6050 4300 30  0001 C CNN
 F 1 "GND" H 6050 4230 30  0001 C CNN
@@
 	6050 4200 6050 4300
 $Comp
-L R R2
+L R-RESCUE-qrpamp R2
 U 1 1 54788FD0
 P 5350 3700
+AR Path="/54788FD0" Ref="R2"  Part="1"
+AR Path="/5470C525/54788FD0" Ref="R2"  Part="1"
 F 0 "R2" V 5430 3700 40  0000 C CNN
 F 1 "680" V 5357 3701 40  0000 C CNN
@@
 $EndComp
 $Comp
-L C C2
+L C-RESCUE-qrpamp C2
 U 1 1 54788FE2
 P 5700 3900
+AR Path="/54788FE2" Ref="C2"  Part="1"
+AR Path="/5470C525/54788FE2" Ref="C2"  Part="1"
 F 0 "C2" H 5700 4000 40  0000 L CNN
 F 1 ".1u" H 5706 3815 40  0000 L CNN
