File: swr.sch (KiCad schematic (older format))
At the start: 8 parts, among them T4 12:1, T5 1:12

Commit message: Update project to kicad bzr 6336
I guess some parts are now outdated
Parts:
- C35, C36: symbol C -> C-RESCUE-qrpamp
- R20, R21: symbol R -> R-RESCUE-qrpamp
Changed lines of the file:
@@
 EESchema Schematic File Version 2
+LIBS:qrpamp-rescue
 LIBS:power
 LIBS:device
@@
 swr_in
 $Comp
-L GND #PWR098
+L GND-RESCUE-qrpamp #PWR098
 U 1 1 54710723
 P 5000 2400
+AR Path="/54710723" Ref="#PWR098"  Part="1"
+AR Path="/5470C635/54710723" Ref="#PWR098"  Part="1"
 F 0 "#PWR098" H 5000 2400 30  0001 C CNN
 F 1 "GND" H 5000 2330 30  0001 C CNN
@@
 swr_gnd
 $Comp
-L GND #PWR099
+L GND-RESCUE-qrpamp #PWR099
 U 1 1 5471074B
 P 4950 3350
+AR Path="/5471074B" Ref="#PWR099"  Part="1"
+AR Path="/5470C635/5471074B" Ref="#PWR099"  Part="1"
 F 0 "#PWR099" H 4950 3350 30  0001 C CNN
 F 1 "GND" H 4950 3280 30  0001 C CNN
@@
 $EndComp
 $Comp
-L GND #PWR0100
+L GND-RESCUE-qrpamp #PWR0100
 U 1 1 5471075F
 P 5350 3650
+AR Path="/5471075F" Ref="#PWR0100"  Part="1"
+AR Path="/5470C635/5471075F" Ref="#PWR0100"  Part="1"
 F 0 "#PWR0100" H 5350 3650 30  0001 C CNN
 F 1 "GND" H 5350 3580 30  0001 C CNN
@@
 	4650 4450 4950 4450
 $Comp
-L R R20
+L R-RESCUE-qrpamp R20
 U 1 1 54710792
 P 4850 4700
+AR Path="/54710792" Ref="R20"  Part="1"
+AR Path="/5470C635/54710792" Ref="R20"  Part="1"
 F 0 "R20" V 4930 4700 40  0000 C CNN
 F 1 "51" V 4857 4701 40  0000 C CNN
@@
 $EndComp
 $Comp
-L R R21
+L R-RESCUE-qrpamp R21
 U 1 1 547107A4
 P 5450 4700
+AR Path="/547107A4" Ref="R21"  Part="1"
+AR Path="/5470C635/547107A4" Ref="R21"  Part="1"
 F 0 "R21" V 5530 4700 40  0000 C CNN
 F 1 "51" V 5457 4701 40  0000 C CNN
@@
 $EndComp
 $Comp
-L GND #PWR0101
+L GND-RESCUE-qrpamp #PWR0101
 U 1 1 54710804
 P 4850 4950
+AR Path="/54710804" Ref="#PWR0101"  Part="1"
+AR Path="/5470C635/54710804" Ref="#PWR0101"  Part="1"
 F 0 "#PWR0101" H 4850 4950 30  0001 C CNN
 F 1 "GND" H 4850 4880 30  0001 C CNN
@@
 $EndComp
 $Comp
-L GND #PWR0102
+L GND-RESCUE-qrpamp #PWR0102
 U 1 1 54710818
 P 5450 4950
+AR Path="/54710818" Ref="#PWR0102"  Part="1"
+AR Path="/5470C635/54710818" Ref="#PWR0102"  Part="1"
 F 0 "#PWR0102" H 5450 4950 30  0001 C CNN
 F 1 "GND" H 5450 4880 30  0001 C CNN
@@
 $EndComp
 $Comp
-L C C36
+L C-RESCUE-qrpamp C36
 U 1 1 5471082C
 P 6050 4250
+AR Path="/5471082C" Ref="C36"  Part="1"
+AR Path="/5470C635/5471082C" Ref="C36"  Part="1"
 F 0 "C36" H 6050 4350 40  0000 L CNN
 F 1 "0.1u" H 6056 4165 40  0000 L CNN
@@
 $EndComp
 $Comp
-L C C35
+L C-RESCUE-qrpamp C35
 U 1 1 5471083E
 P 4250 4250
+AR Path="/5471083E" Ref="C35"  Part="1"
+AR Path="/5470C635/5471083E" Ref="C35"  Part="1"
 F 0 "C35" H 4250 4350 40  0000 L CNN
 F 1 "0.1u" H 4256 4165 40  0000 L CNN
@@
 $EndComp
 $Comp
-L GND #PWR0103
+L GND-RESCUE-qrpamp #PWR0103
 U 1 1 5471084B
 P 4250 4050
+AR Path="/5471084B" Ref="#PWR0103"  Part="1"
+AR Path="/5470C635/5471084B" Ref="#PWR0103"  Part="1"
 F 0 "#PWR0103" H 4250 4050 30  0001 C CNN
 F 1 "GND" H 4250 3980 30  0001 C CNN
@@
 $EndComp
 $Comp
-L GND #PWR0104
+L GND-RESCUE-qrpamp #PWR0104
 U 1 1 54710867
 P 6050 4050
+AR Path="/54710867" Ref="#PWR0104"  Part="1"
+AR Path="/5470C635/54710867" Ref="#PWR0104"  Part="1"
 F 0 "#PWR0104" H 6050 4050 30  0001 C CNN
 F 1 "GND" H 6050 3980 30  0001 C CNN
